File: MT7620N.kicad_pcb (KiCad board)
At the start: 2 copper layers, 146 x 127 mm, 176 parts, among them J1 POWERJACK-DC21_2, P2 IO_HOLE-3.2-BIG, P6 IO_HOLE-3.2-BIG, P7 IO_HOLE-3.2-BIG, P8 IO_HOLE-3.2-BIG, Q1 2N3904, Q2 2N3904, U1 IC_MP1484EN_SOIC08, U10 DLW21SN900SQ2, U11 IP4220CZ6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

Commit message: 完成新要求修改，生成gerber文件
Parts:
- C23, C24, R21: moved to B.Cu
- C25, C29, L10, L11, L14, L15, L6, L7: moved to F.Cu
- U20, U21: footprint IO_RJ45X1 -> IO_RJ45X1-8P8C-90
- X1: footprint C_CRY_5.0-3.2 -> C_CRY_DIP2
- moved U11 51.1 mm to (130.6, 186.7), turned to 0 degrees
- moved U5 47.3 mm to (130.8, 182.9), turned to 0 degrees
- moved U13 33.8 mm to (156.0, 186.6), turned to 0 degrees
- moved U9 30.5 mm to (156.2, 182.9), turned to 0 degrees
- moved L14 15.5 mm to (135.9, 184.2), turned to 180 degrees
- moved L15 15.5 mm to (161.3, 184.2), turned to 180 degrees
- moved C29 10.2 mm to (125.7, 184.2)
- moved C25 9.99 mm to (151.1, 184.4)
- moved L7 9.03 mm to (161.3, 186.7), turned to 180 degrees
- moved L11 9.03 mm to (135.9, 186.7), turned to 180 degrees
- moved L10 7.24 mm to (125.7, 186.7), turned to 0 degrees
- moved L6 7.24 mm to (151.1, 186.7), turned to 0 degrees
- moved U20 6.84 mm to (104.1, 192.4)
- moved C23 6.71 mm to (184.8, 140.3), turned to 90 degrees
- moved R21 5.09 mm to (154.6, 109.6), turned to 180 degrees
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Routing:
- net +5V: track 82.8 -> 676.3 mm, vias 1 -> 109
- net +3.3V: track 125.4 -> 496.8 mm, vias 13 -> 22
- net /I2C_SD: track 0.00 -> 209.0 mm
- net /LINK4: track 0.00 -> 191.6 mm
- net /LINK1: track 0.00 -> 190.2 mm
- net /LINK0: track 0.00 -> 188.5 mm
- net GND: track 175.3 -> 355.3 mm, vias 36 -> 47
- net /SATA/TXN: track 0.00 -> 135.8 mm, vias 0 -> 1
- net /SATA/TXP: track 0.00 -> 134.6 mm, vias 0 -> 1
- net /I2C_SCLK: track 0.00 -> 129.0 mm
- net /GPIO0: track 0.00 -> 128.2 mm
- net /ANT_TRNB: track 0.00 -> 128.1 mm
- net /WDT_RST_N: track 0.00 -> 124.6 mm
- net /LINK2: track 0.00 -> 123.3 mm
- net /ANT_TRN: track 1.88 -> 125.0 mm
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- added copper zone on F.Cu, net +3.3V
- added copper zone on B.Cu, net +5V
- added copper zone on F.Cu, net +5V
- added copper zone on B.Cu, net GND
- added copper zone on F.Cu, net GND
- added copper zone on F.Cu, net N-00000173
- added copper zone on F.Cu, net N-00000174
Other:
- board text added: "3.3V"
- board text added: "ANT_TRN/IO=19"
- board text added: "ANT_TRNB/IO=18"
- board text added: "EPHY 0"
- board text added: "EPHY 1"
- board text added: "EPHY 2"
- board text added: "EPHY 3"
- board text added: "EPHY 4"
- board text added: "EPHY_LED0/IO=40"
- board text added: "EPHY_LED1/IO=41"
- board text added: "EPHY_LED2/IO=42"
- board text added: "EPHY_LED3/IO=43"
- board text added: "EPHY_LED4/IO=44"
- board text added: "GND"
- board text added: "GPIO"
- board text added: "GPIO0/O=0"
- board text added: "I2C_SCLK/IO=2"
- board text added: "I2C_SD/IO=1"
- board text added: "PA_PE_G0/IO=20"
- board text added: "PA_PE_G1/IO=21"
- board text added: "VBUS"
- board text added: "WDT_RST_N/IO=17"
- board text added: "WLED_N/IO=72"
- board text removed: "+"
- board text removed: "-"
- board text removed: "ANT_TRN"
- board text removed: "ANT_TRNB"
- board text removed: "EPHY_LED0"
- board text removed: "EPHY_LED1"
- board text removed: "EPHY_LED2"
- board text removed: "EPHY_LED3"
- board text removed: "EPHY_LED4"
- board text removed: "GPIO0"
- board text removed: "I2C_SCLK"
- board text removed: "LAN"
- board text removed: "PA_PE_G0"
- board text removed: "PA_PE_G1"
- board text removed: "PORT2"
- board text removed: "PORT3"
- board text removed: "PORT4"
- board text removed: "S"
- board text removed: "WAN"
- board text removed: "WDT_RST_N"
- board text removed: "WLED_N"
- board text removed: "W_I2C_SD"
