File: MT7620N.sch (KiCad schematic (older format))
At the start: 45 parts, among them P1 IO_HOLE-3.2-BIG, P2 IO_HOLE-3.2-BIG, P3 IO_HOLE-3.2-BIG, P4 IO_HOLE-3.2-BIG, P5 IO_HOLE-3.2-BIG, P6 IO_HOLE-3.2-BIG, P7 IO_HOLE-3.2-BIG, P8 IO_HOLE-3.2-BIG

Commit message: 新修改布局
Parts:
- removed JP10, JP11, JP12, JP13, JP14, JP17, JP18, JP22, JP24, JP25, JP28, JP30, JP31, JP32, JP33, JP4, JP5, JP6, JP9: IO_M03X1, IO_M03X1, symbol IO_M03X1
- removed P1, P2, P3, P4, P5, P6, P7, P8: IO_HOLE-3.2-BIG, IO_HOLE-3.2-big, symbol IO_HOLE-3.2-BIG
- added JP10: IO_M03X2, -CON-PANDUIT_057-006-1, symbol IO_M03X2
- added JP3: IO_M03X1, IO_M03X1, symbol IO_M03X1
- added JP4, JP5, JP6: IO_M04X1, IO_M04X1, symbol IO_M04X1
Connections:
- wire segments 240 -> 170
Other:
- moved on the sheet: JP15, JP16, JP21, JP23, JP29, JP38, JP39
