File: WLAN.sch (KiCad schematic (older format))
At the start: 10 parts, among them U20 IO_RJ45X1-JACK, U21 IO_RJ45X1-JACK, U6 HN2066CG_DIP20

Commit message: 完成新要求修改，生成gerber文件
Parts:
- U20, U21: footprint IO_RJ45X1 -> IO_RJ45X1-8P8C-90
Changed lines of the file:
@@
-EESchema Schematic File Version 2  date 2014/12/30 17:10:49
+EESchema Schematic File Version 2  date 2015/1/4 11:31:27
 LIBS:C
 LIBS:IC
@@
 Sheet 5 5
 Title ""
-Date "30 dec 2014"
+Date "4 jan 2015"
 Rev ""
 Comp ""
@@
 F 0 "U20" H 8600 2300 60  0000 C CNN
 F 1 "IO_RJ45X1-JACK" H 8600 2150 60  0000 C CNN
-F 2 "IO_RJ45X1" H 8600 1750 60  0001 C CNN
+F 2 "IO_RJ45X1-8P8C-90" H 8600 1750 60  0001 C CNN
 F 3 "" H 8600 1750 60  0000 C CNN
 	1    8600 1750
@@
 F 0 "U21" H 8600 3050 60  0000 C CNN
 F 1 "IO_RJ45X1-JACK" H 8600 2900 60  0000 C CNN
-F 2 "IO_RJ45X1" H 8600 2500 60  0001 C CNN
+F 2 "IO_RJ45X1-8P8C-90" H 8600 2500 60  0001 C CNN
 F 3 "" H 8600 2500 60  0000 C CNN
 	1    8600 2500
