File: hardware/accessaries/LED/LED.sch (KiCad schematic (older format))
At the start: 16 parts, among them P1 IO_HOLE-3.2, P2 IO_HOLE-3.2, P3 IO_HOLE-3.2, P4 IO_HOLE-3.2, P5 IO_HOLE-3.2, P6 IO_HOLE-3.2, P7 IO_HOLE-3.2, P8 IO_HOLE-3.2

Commit message: Separate into two modules
Parts:
- removed D1: C_DIODE-1N4148_MINIMELF, C_DIODE-1N4148_MINIMELF, symbol C_DIODE-1N4148_MINIMELF
- removed JP2: IO_MOLEX_70554-03, IO_MOLEX_70554-03, symbol IO_MOLEX_70554-03
- removed P5, P6, P7, P8: IO_HOLE-3.2, IO_HOLE-3.2, symbol IO_HOLE-3.2
- removed R2: 4.7K, C_R_0805, symbol C_R_0805
- removed S1: C_SW_OMRON-10-XX, switch-omron-B3F-40XX, symbol C_SW_OMRON-10-XX
Connections:
- wire segments 25 -> 10
Changed lines of the file:
@@
-EESchema Schematic File Version 2  date 2015/1/6 10:04:06
+EESchema Schematic File Version 2
 LIBS:power
 LIBS:device
@@
 LIBS:contrib
 LIBS:valves
-LIBS:C
-LIBS:IC
-LIBS:I-O
-LIBS:rcl
 LIBS:LED-cache
 EELAYER 27 0
@@
 Sheet 1 1
 Title ""
-Date "6 jan 2015"
+Date "26 feb 2015"
 Rev ""
 Comp ""
@@
 $EndComp
 $Comp
-L IO_MOLEX_70554-03 JP2
-U 1 1 54A90BB9
-P 3650 6150
-F 0 "JP2" H 3450 5880 50  0000 L BNN
-F 1 "IO_MOLEX_70554-03" H 2400 6100 50  0000 L BNN
-F 2 "IO_MOLEX_70554-03" H 3400 6400 50  0001 C CNN
-F 3 "~" H 3650 6150 60  0000 C CNN
-	1    3650 6150
-	1    0    0    1
-$EndComp
-$Comp
-L GND #PWR2
-U 1 1 54A90BBF
-P 3900 6850
-F 0 "#PWR2" H 3900 6850 30  0001 C CNN
-F 1 "GND" H 3900 6780 30  0001 C CNN
-F 2 "" H 3900 6850 60  0000 C CNN
-F 3 "" H 3900 6850 60  0000 C CNN
-	1    3900 6850
-	1    0    0    -1
-$EndComp
-Wire Wire Line
-	3800 6050 3900 6050
-Wire Wire Line
-	3900 6050 3900 6850
-Wire Wire Line
-	4000 5550 4000 6150
-Wire Wire Line
-	3800 6250 4950 6250
-$Comp
-L C_SW_OMRON-10-XX S1
-U 1 1 54A90C06
-P 5150 6250
-F 0 "S1" V 5065 6450 50  0000 L BNN
-F 1 "C_SW_OMRON-10-XX" V 5450 5950 50  0001 L BNN
-F 2 "switch-omron-B3F-40XX" H 5200 5900 50  0001 C CNN
-F 3 "~" H 5150 6250 60  0000 C CNN
-	1    5150 6250
-	0    -1   -1   0
-$EndComp
-$Comp
-L C_R_0805 R2
-U 1 1 54A90C6A
-P 4450 5900
-F 0 "R2" H 4400 5959 50  0000 L BNN
-F 1 "4.7K" H 4400 5750 50  0000 L BNN
-F 2 "C_R_0805" H 4450 6050 50  0001 C CNN
-F 3 "~" H 4450 5900 60  0000 C CNN
-	1    4450 5900
-	0    -1   -1   0
-$EndComp
-$Comp
-L GND #PWR7
-U 1 1 54A90CD2
-P 5550 6650
-F 0 "#PWR7" H 5550 6650 30  0001 C CNN
-F 1 "GND" H 5550 6580 30  0001 C CNN
-F 2 "" H 5550 6650 60  0000 C CNN
-F 3 "" H 5550 6650 60  0000 C CNN
-	1    5550 6650
-	1    0    0    -1
-$EndComp
-$Comp
-L IO_HOLE-3.2 P5
-U 1 1 54A90CF8
-P 7900 5400
-F 0 "P5" H 7900 5600 60  0001 C CNN
-F 1 "IO_HOLE-3.2" H 7900 5400 60  0001 C CNN
-F 2 "IO_HOLE-3.2" H 7900 5200 60  0001 C CNN
-F 3 "~" H 7900 5400 60  0000 C CNN
-	1    7900 5400
-	1    0    0    -1
-$EndComp
-$Comp
-L IO_HOLE-3.2 P6
-U 1 1 54A90CFE
-P 8300 5400
-F 0 "P6" H 8300 5600 60  0001 C CNN
-F 1 "IO_HOLE-3.2" H 8300 5400 60  0001 C CNN
-F 2 "IO_HOLE-3.2" H 8300 5200 60  0001 C CNN
-F 3 "~" H 8300 5400 60  0000 C CNN
-	1    8300 5400
-	1    0    0    -1
-$EndComp
-$Comp
-L IO_HOLE-3.2 P7
-U 1 1 54A90D04
-P 8700 5400
-F 0 "P7" H 8700 5600 60  0001 C CNN
-F 1 "IO_HOLE-3.2" H 8700 5400 60  0001 C CNN
-F 2 "IO_HOLE-3.2" H 8700 5200 60  0001 C CNN
-F 3 "~" H 8700 5400 60  0000 C CNN
-	1    8700 5400
-	1    0    0    -1
-$EndComp
-$Comp
-L IO_HOLE-3.2 P8
-U 1 1 54A90D0A
-P 9100 5400
-F 0 "P8" H 9100 5600 60  0001 C CNN
-F 1 "IO_HOLE-3.2" H 9100 5400 60  0001 C CNN
-F 2 "IO_HOLE-3.2" H 9100 5200 60  0001 C CNN
-F 3 "~" H 9100 5400 60  0000 C CNN
-	1    9100 5400
-	1    0    0    -1
-$EndComp
-$Comp
 L +3.3V #PWR3
 U 1 1 54AB39B4
@@
 F 3 "~" H 4000 3250 60  0000 C CNN
 	1    4000 3250
-	1    0    0    -1
-$EndComp
-$Comp
-L +3.3V #PWR4
-U 1 1 54AB39D5
-P 4000 5550
-F 0 "#PWR4" H 4000 5660 30  0001 C CNN
-F 1 "+3.3V" H 4000 5660 30  0000 C CNN
-F 2 "~" H 4000 5550 60  0000 C CNN
-F 3 "~" H 4000 5550 60  0000 C CNN
-	1    4000 5550
 	1    0    0    -1
 $EndComp
@@
 	1    0    0    -1
 $EndComp
-Wire Wire Line
-	4000 6150 3800 6150
-$Comp
-L C_DIODE-1N4148_MINIMELF D1
-U 1 1 54AB3B64
-P 4700 5900
-F 0 "D1" H 4650 5769 50  0000 L BNN
-F 1 "C_DIODE-1N4148_MINIMELF" H 4200 5659 50  0001 L BNN
-F 2 "C_DIODE-1N4148_MINIMELF" H 4700 6050 50  0001 C CNN
-F 3 "~" H 4700 5900 60  0000 C CNN
-	1    4700 5900
-	0    -1   -1   0
-$EndComp
-Wire Wire Line
-	4450 6250 4450 6100
-Wire Wire Line
-	4700 6250 4700 6050
-Connection ~ 4450 6250
-$Comp
-L +3.3V #PWR6
-U 1 1 54AB3CDC
-P 4450 5550
-F 0 "#PWR6" H 4450 5660 30  0001 C CNN
-F 1 "+3.3V" H 4450 5660 30  0000 C CNN
-F 2 "~" H 4450 5550 60  0000 C CNN
-F 3 "~" H 4450 5550 60  0000 C CNN
-	1    4450 5550
-	1    0    0    -1
-$EndComp
-Wire Wire Line
-	4450 5700 4450 5550
-Wire Wire Line
-	4700 5750 4700 5600
-Wire Wire Line
-	4700 5600 4450 5600
-Connection ~ 4450 5600
-Connection ~ 4700 6250
-Wire Wire Line
-	4950 6150 4850 6150
-Wire Wire Line
-	4850 6150 4850 6250
-Connection ~ 4850 6250
-Wire Wire Line
-	5350 6150 5550 6150
-Wire Wire Line
-	5550 6150 5550 6650
-Wire Wire Line
-	5350 6250 5550 6250
-Connection ~ 5550 6250
 $Comp
 L C_LED_LED5MM LED1
